Commit message: xarm6 description

File: src/robot_descriptions/xarm6/urdf/xarm6_robot.urdf (robot description, URDF)
Before this commit: robot xarm6, 8 links, 7 joints
Links:
- link link1: geometry collision mesh filename=package://xarm6/meshes/collision/link1_vhacd.obj; visual mesh filename=package://xarm6/meshes/visual/link1.stl
- link link2: geometry collision mesh filename=package://xarm6/meshes/collision/link2_vhacd.obj; visual mesh filename=package://xarm6/meshes/visual/link2.stl
- link link3: geometry collision mesh filename=package://xarm6/meshes/collision/link3_vhacd.obj; visual mesh filename=package://xarm6/meshes/visual/link3.stl
- link link4: geometry collision mesh filename=package://xarm6/meshes/collision/link4_vhacd.obj; visual mesh filename=package://xarm6/meshes/visual/link4.stl
- link link5: geometry collision mesh filename=package://xarm6/meshes/collision/link5_vhacd.obj; visual mesh filename=package://xarm6/meshes/visual/link5.stl
- link link6: geometry collision mesh filename=package://xarm6/meshes/collision/link6_vhacd.obj; visual mesh filename=package://xarm6/meshes/visual/link6.stl
- link link_base: geometry collision mesh filename=package://xarm6/meshes/collision/base_vhacd.obj; visual mesh filename=package://xarm6/meshes/visual/base.stl
