Commit message: xarm6

File: src/robot_descriptions/xarm6/urdf/xarm6.urdf.xacro (robot description, xacro)
@@ -1,20 +1,30 @@
 <?xml version="1.0"?>
 <robot xmlns:xacro="http://ros.org/wiki/xacro">
-  <xacro:macro name="lite6_urdf" params="prefix
+  <xacro:macro name="xarm6_urdf" params="prefix
     joint1_lower_limit:=${-2.0*pi}  joint1_upper_limit:=${2.0*pi}
-    joint2_lower_limit:=${-2.61799}  joint2_upper_limit:=${2.61799}
-    joint3_lower_limit:=${-0.061087}  joint3_upper_limit:=${5.235988}
+    joint2_lower_limit:=${-2.059}  joint2_upper_limit:=${2.0944}
+    joint3_lower_limit:=${-3.927}  joint3_upper_limit:=${0.19198}
     joint4_lower_limit:=${-2.0*pi}  joint4_upper_limit:=${2.0*pi}
-    joint5_lower_limit:=${-2.1642}  joint5_upper_limit:=${2.1642}
+    joint5_lower_limit:=${-1.69297}  joint5_upper_limit:=${pi}
     joint6_lower_limit:=${-2.0*pi}  joint6_upper_limit:=${2.0*pi}
+    model1300:=false
     inertial_params_filename:='' kinematics_params_filename:='' "
     >
+    <!-- define property -->
+    <xacro:if value="${model1300}">
+      <xacro:property name="end_tool_visual_filename" value="end_tool/visual/end_tool_1300"/>
+      <xacro:property name="end_tool_collision_filename" value="end_tool/collision/end_tool_1300"/>
+    </xacro:if>
+    <xacro:unless value="${model1300}">
+      <xacro:property name="end_tool_visual_filename" value="xarm6/visual/link6"/>
+      <xacro:property name="end_tool_collision_filename" value="end_tool/collision/end_tool"/>
+    </xacro:unless>
     <!-- load params and define property -->
-    <xacro:property name="default_inertial_params_filename" value="xarm6_type9_HT_BR2"/>
+    <xacro:property name="default_inertial_params_filename" value="xarm6_type6_HT_BR2"/>
     <xacro:if value="${inertial_params_filename != ''}">
-      <xacro:property name="link_inertial_params_file" value="$(find xarm_description)/config/link_inertial/${inertial_params_filename}.yaml"/>
+      <xacro:property name="link_inertial_params_file" value="$(find xarm6)/config/link_inertial/${inertial_params_filename}.yaml"/>
     </xacro:if>
     <xacro:unless value="${inertial_params_filename != ''}">
-      <xacro:property name="link_inertial_params_file" value="$(find xarm_description)/config/link_inertial/${default_inertial_params_filename}.yaml"/>
+      <xacro:property name="link_inertial_params_file" value="$(find xarm6)/config/link_inertial/${default_inertial_params_filename}.yaml"/>
     </xacro:unless>
     <xacro:if value="${use_xacro_load_yaml}">
@@ -29,17 +39,17 @@
     <link name="${prefix}link_base">
       <inertial>
-        <origin xyz="-0.00829544579053192 3.26357432323433E-05 0.0631194584987089" rpy="0 0 0" />
-        <mass value="1.65393501783165" />
+        <origin xyz="0.0 0.0 0.09103" rpy="0 0 0" />
+        <mass value="2.7" />
         <inertia
-          ixx="0" ixy="0" ixz="0"
-          iyy="0" iyz="0" izz="0" />
+          ixx="0.00494875" ixy="-3.5E-06" ixz="1.25E-05"
+          iyy="0.00494174" iyz="1.67E-06" izz="0.002219" />
       </inertial>
       <xacro:common_link_visual
-        mesh_filename="lite6/visual/link_base"
-        origin_xyz="0 0 0"
-        origin_rpy="0 0 0"
-        material_name="${prefix}White" />
-      <xacro:common_link_collision
-        mesh_filename="lite6/collision/link_base"
+        mesh_filename="xarm6/visual/link_base"
+        origin_xyz="0 0 0"
+        origin_rpy="0 0 0"
+        material_name="${prefix}White" />
+      <xacro:common_link_collision
+        mesh_filename="xarm6/visual/link_base"
         origin_xyz="0 0 0"
         origin_rpy="0 0 0" />
@@ -50,19 +60,19 @@
         origin_rpy="0 0 0"/>
       <xacro:common_link_visual
-        mesh_filename="lite6/visual/link1"
-        origin_xyz="0 0 0"
-        origin_rpy="0 0 0"
-        material_name="${prefix}White" />
-      <xacro:common_link_collision
-        mesh_filename="lite6/collision/link1"
+        mesh_filename="xarm6/visual/link1"
+        origin_xyz="0 0 0"
+        origin_rpy="0 0 0"
+        material_name="${prefix}White" />
+      <xacro:common_link_collision
+        mesh_filename="xarm6/visual/link1"
         origin_xyz="0 0 0"
         origin_rpy="0 0 0" />
     </link>
     <joint name="${prefix}joint1" type="revolute">
-      <!-- <origin xyz="0 0 0.2435" rpy="0 0 0" /> -->
+      <parent link="${prefix}link_base"/>
+      <child link="${prefix}link1"/>
+      <!-- <origin xyz="0 0 0.267" rpy="0 0 0"/> -->
       <xacro:common_joint_origin joint_kinematic_params="${kinematics_params['joint1']}" />
-      <parent link="${prefix}link_base" />
-      <child link="${prefix}link1" />
-      <axis xyz="0 0 1" />
+      <axis xyz="0 0 1"/>
       <limit
         lower="${joint1_lower_limit}"
@@ -77,19 +87,19 @@
         origin_rpy="0 0 0"/>
       <xacro:common_link_visual
-        mesh_filename="lite6/visual/link2"
+        mesh_filename="xarm6/visual/link2"
         origin_xyz="0 0 ${-kinematics_params['joint2']['y']}"
         origin_rpy="0 0 0"
         material_name="${prefix}White" />
       <xacro:common_link_collision
-        mesh_filename="lite6/collision/link2"
+        mesh_filename="xarm6/visual/link2"
         origin_xyz="0 0 ${-kinematics_params['joint2']['y']}"
         origin_rpy="0 0 0" />
     </link>
     <joint name="${prefix}joint2" type="revolute">
-      <!-- <origin xyz="0 0 0" rpy="1.5708 -1.5708 3.1416" /> -->
+      <parent link="${prefix}link1"/>
+      <child link="${prefix}link2"/>
+      <!-- <origin xyz="0 0 0" rpy="-1.5708 0 0" /> -->
       <xacro:common_joint_origin joint_kinematic_params="${kinematics_params['joint2']}" />
-      <parent link="${prefix}link1" />
-      <child link="${prefix}link2" />
-      <axis xyz="0 0 1" />
+      <axis xyz="0 0 1"/>
       <limit
         lower="${joint2_lower_limit}"
@@ -104,19 +114,19 @@
         origin_rpy="0 0 0"/>
       <xacro:common_link_visual
-        mesh_filename="lite6/visual/link3"
-        origin_xyz="0 0 0"
-        origin_rpy="0 0 0"
-        material_name="${prefix}White" />
-      <xacro:common_link_collision
-        mesh_filename="lite6/collision/link3"
+        mesh_filename="xarm6/visual/link3"
+        origin_xyz="0 0 0"
+        origin_rpy="0 0 0"
+        material_name="${prefix}White" />
+      <xacro:common_link_collision
+        mesh_filename="xarm6/visual/link3"
         origin_xyz="0 0 0"
         origin_rpy="0 0 0" />
     </link>
     <joint name="${prefix}joint3" type="revolute">
-      <!-- <origin xyz="0.2002 0 0" rpy="-3.1416 0 1.5708" /> -->
+      <parent link="${prefix}link2"/>
+      <child link="${prefix}link3"/>
+      <!-- <origin xyz="0.0535 -0.2845 0" rpy="0 0 0"/> -->
       <xacro:common_joint_origin joint_kinematic_params="${kinematics_params['joint3']}" />
-      <parent link="${prefix}link2" />
-      <child link="${prefix}link3" />
-      <axis xyz="0 0 1" />
+      <axis xyz="0 0 1"/>
       <limit
         lower="${joint3_lower_limit}"
@@ -131,19 +141,19 @@
         origin_rpy="0 0 0"/>
       <xacro:common_link_visual
-        mesh_filename="lite6/visual/link4"
-        origin_xyz="0 0 0"
-        origin_rpy="0 0 0"
-        material_name="${prefix}White" />
-      <xacro:common_link_collision
-        mesh_filename="lite6/collision/link4"
+        mesh_filename="xarm6/visual/link4"
+        origin_xyz="0 0 0"
+        origin_rpy="0 0 0"
+        material_name="${prefix}White" />
+      <xacro:common_link_collision
+        mesh_filename="xarm6/visual/link4"
         origin_xyz="0 0 0"
         origin_rpy="0 0 0" />
     </link>
     <joint name="${prefix}joint4" type="revolute">
-      <!-- <origin xyz="0.087 -0.22761 0" rpy="1.5708 0 0" /> -->
+      <parent link="${prefix}link3"/>
+      <child link="${prefix}link4"/>
+      <!-- <origin xyz="0.0775 0.3425 0" rpy="-1.5708 0 0"/> -->
       <xacro:common_joint_origin joint_kinematic_params="${kinematics_params['joint4']}" />
-      <parent link="${prefix}link3" />
-      <child link="${prefix}link4" />
-      <axis xyz="0 0 1" />
+      <axis xyz="0 0 1"/>
       <limit
         lower="${joint4_lower_limit}"
@@ -158,19 +168,18 @@
         origin_rpy="0 0 0"/>
       <xacro:common_link_visual
-        mesh_filename="lite6/visual/link5"
-        origin_xyz="0 0 0"
-        origin_rpy="0 0 0"
-        material_name="${prefix}White" />
-      <xacro:common_link_collision
-        mesh_filename="lite6/collision/link5"
+        mesh_filename="xarm6/visual/link5"
+        origin_xyz="0 0 0"
+        origin_rpy="0 0 0"
+        material_name="${prefix}White" />
+      <xacro:common_link_collision
+        mesh_filename="xarm6/visual/link5"
         origin_xyz="0 0 0"
         origin_rpy="0 0 0" />
     </link>
     <joint name="${prefix}joint5" type="revolute">
-      <!-- <origin xyz="0 0 0" rpy="1.5708 0 0" /> -->
+      <parent link="${prefix}link4"/>
+      <child link="${prefix}link5"/>
       <xacro:common_joint_origin joint_kinematic_params="${kinematics_params['joint5']}" />
-      <parent link="${prefix}link4" />
-      <child link="${prefix}link5" />
-      <axis xyz="0 0 1" />
+      <axis xyz="0 0 1"/>
       <limit
         lower="${joint5_lower_limit}"
@@ -185,19 +194,19 @@
         origin_rpy="0 0 0"/>
       <xacro:common_link_visual
-        mesh_filename="lite6/visual/link6"
+        mesh_filename="${end_tool_visual_filename}"
         origin_xyz="0 0 0"
         origin_rpy="0 0 0"
         material_name="${prefix}Silver" />
       <xacro:common_link_collision
-        mesh_filename="lite6/collision/link6"
+        mesh_filename="${end_tool_collision_filename}"
         origin_xyz="0 0 0"
         origin_rpy="0 0 0" />
     </link>
     <joint name="${prefix}joint6" type="revolute">
-      <!-- <origin xyz="0 0.0625 0" rpy="-1.5708 0 0" /> -->
+      <parent link="${prefix}link5"/>
+      <child link="${prefix}link6"/>
+      <!-- <origin xyz="0.076 0.097 0" rpy="-1.5708 0 0"/> -->
       <xacro:common_joint_origin joint_kinematic_params="${kinematics_params['joint6']}" />
-      <parent link="${prefix}link5" />
-      <child link="${prefix}link6" />
-      <axis xyz="0 0 1" />
+      <axis xyz="0 0 1"/>
       <limit
         lower="${joint6_lower_limit}"
