Commit message: replacing

File: src/robot_descriptions/xarm6_description/urdf/dual_xarm_device.urdf.xacro (robot description, xacro)
@@ -63,5 +63,5 @@
   <xacro:arg name="kinematics_suffix_2" default=""/>
   <!-- load xarm device -->
-  <xacro:include filename="$(find xarm_description)/urdf/xarm_device_macro.xacro" />
+  <xacro:include filename="$(find xarm6_description)/urdf/xarm_device_macro.xacro" />
   <xacro:xarm_device prefix="$(arg prefix_1)" hw_ns="$(arg hw_ns)" limited="$(arg limited)"
     effort_control="$(arg effort_control)" velocity_control="$(arg velocity_control)"

File: src/robot_descriptions/xarm6_description/urdf/gripper/bio_gripper_macro.xacro (robot description, xacro)
@@ -2,8 +2,8 @@
 <robot xmlns:xacro="http://ros.org/wiki/xacro" name="xarm_gripper" >
   <!-- xarm_gripper -->
-  <xacro:include filename="$(find xarm_description)/urdf/gripper/bio_gripper.ros2_control.xacro" />
-  <xacro:include filename="$(find xarm_description)/urdf/gripper/bio_gripper.urdf.xacro" />
-  <xacro:include filename="$(find xarm_description)/urdf/gripper/bio_gripper.transmission.xacro" />
-  <xacro:include filename="$(find xarm_description)/urdf/gripper/bio_gripper.gazebo.xacro" />
+  <xacro:include filename="$(find xarm6_description)/urdf/gripper/bio_gripper.ros2_control.xacro" />
+  <xacro:include filename="$(find xarm6_description)/urdf/gripper/bio_gripper.urdf.xacro" />
+  <xacro:include filename="$(find xarm6_description)/urdf/gripper/bio_gripper.transmission.xacro" />
+  <xacro:include filename="$(find xarm6_description)/urdf/gripper/bio_gripper.gazebo.xacro" />
   <xacro:macro name="bio_gripper_macro" params="prefix:='' attach_to:='' ns:='xarm' attach_xyz:='0 0 0' attach_rpy:='0 0 0'
     ros2_control_plugin:='uf_robot_hardware/UFRobotFakeSystemHardware' dof:=7 hard_interface:='PositionJointInterface' ">

File: src/robot_descriptions/xarm6_description/urdf/gripper/gripper.urdf.xacro (robot description, xacro)
@@ -4,5 +4,5 @@
   <xacro:arg name="prefix" default=""/>
   <xacro:arg name="mesh_suffix" default="stl"/>
-  <xacro:include filename="$(find xarm_description)/urdf/gripper/gripper_macro.xacro" />
+  <xacro:include filename="$(find xarm6_description)/urdf/gripper/gripper_macro.xacro" />
   <xacro:gripper_device robot_type="$(arg robot_type)" prefix="$(arg prefix)" mesh_suffix="$(arg mesh_suffix)" />
 </robot>

File: src/robot_descriptions/xarm6_description/urdf/gripper/gripper_macro.xacro (robot description, xacro)
@@ -3,25 +3,25 @@
   <xacro:macro name="gripper_device" params="prefix:='' robot_type:='xarm' mesh_suffix:='stl' ">
     <!-- Load Common Material -->
-    <xacro:include filename="$(find xarm_description)/urdf/_private_macro.xacro" />
+    <xacro:include filename="$(find xarm6_description)/urdf/_private_macro.xacro" />
     <xacro:device_macro_begin />
     <!-- Load Common Material -->
-    <xacro:include filename="$(find xarm_description)/urdf/common/common.material.xacro" />
+    <xacro:include filename="$(find xarm6_description)/urdf/common/common.material.xacro" />
     <xacro:common_material prefix="${prefix}"/>
-    <xacro:property name="mesh_path" value="package://xarm_description/meshes" scope="parent"/>
+    <xacro:property name="mesh_path" value="package://xarm6_description/meshes" scope="parent"/>
     <!-- include common.link.xacro -->
-    <xacro:include filename="$(find xarm_description)/urdf/common/common.link.xacro" />
+    <xacro:include filename="$(find xarm6_description)/urdf/common/common.link.xacro" />
     <xacro:if value="${robot_type == 'lite'}">
       <!-- Load Lite Gripper Model URDF -->
-      <xacro:include filename="$(find xarm_description)/urdf/gripper/lite_gripper.urdf.xacro" />
+      <xacro:include filename="$(find xarm6_description)/urdf/gripper/lite_gripper.urdf.xacro" />
       <xacro:uflite_gripper_urdf prefix="${prefix}" />
     </xacro:if>
     <xacro:if value="${robot_type == 'bio'}">
       <!-- Load BIO Gripper Model URDF -->
-      <xacro:include filename="$(find xarm_description)/urdf/gripper/bio_gripper_macro.xacro" />
+      <xacro:include filename="$(find xarm6_description)/urdf/gripper/bio_gripper_macro.xacro" />
       <xacro:bio_gripper_macro prefix="${prefix}" />
     </xacro:if>
     <xacro:unless value="${robot_type == 'lite' or robot_type == 'bio'}">
       <!-- Load XArm Gripper Model URDF -->
-      <xacro:include filename="$(find xarm_description)/urdf/gripper/xarm_gripper_macro.xacro" />
+      <xacro:include filename="$(find xarm6_description)/urdf/gripper/xarm_gripper_macro.xacro" />
       <xacro:xarm_gripper_macro prefix="${prefix}" />
     </xacro:unless>

File: src/robot_descriptions/xarm6_description/urdf/gripper/xarm_gripper_macro.xacro (robot description, xacro)
@@ -2,8 +2,8 @@
 <robot xmlns:xacro="http://ros.org/wiki/xacro" name="xarm_gripper" >
   <!-- xarm_gripper -->
-  <xacro:include filename="$(find xarm_description)/urdf/gripper/xarm_gripper.ros2_control.xacro" />
-  <xacro:include filename="$(find xarm_description)/urdf/gripper/xarm_gripper.urdf.xacro" />
-  <xacro:include filename="$(find xarm_description)/urdf/gripper/xarm_gripper.transmission.xacro" />
-  <xacro:include filename="$(find xarm_description)/urdf/gripper/xarm_gripper.gazebo.xacro" />
+  <xacro:include filename="$(find xarm6_description)/urdf/gripper/xarm_gripper.ros2_control.xacro" />
+  <xacro:include filename="$(find xarm6_description)/urdf/gripper/xarm_gripper.urdf.xacro" />
+  <xacro:include filename="$(find xarm6_description)/urdf/gripper/xarm_gripper.transmission.xacro" />
+  <xacro:include filename="$(find xarm6_description)/urdf/gripper/xarm_gripper.gazebo.xacro" />
   <xacro:macro name="xarm_gripper_macro" params="prefix:='' attach_to:='' ns:='xarm' attach_xyz:='0 0 0' attach_rpy:='0 0 0'
     ros2_control_plugin:='uf_robot_hardware/UFRobotFakeSystemHardware' dof:=7 hard_interface:='PositionJointInterface' ">

File: src/robot_descriptions/xarm6_description/urdf/lite6/lite6.urdf.xacro (robot description, xacro)
@@ -13,8 +13,8 @@
     <xacro:property name="default_inertial_params_filename" value="xarm6_type9_HT_BR2"/>
     <xacro:if value="${inertial_params_filename != ''}">
-      <xacro:property name="link_inertial_params_file" value="$(find xarm_description)/config/link_inertial/${inertial_params_filename}.yaml"/>
+      <xacro:property name="link_inertial_params_file" value="$(find xarm6_description)/config/link_inertial/${inertial_params_filename}.yaml"/>
     </xacro:if>
     <xacro:unless value="${inertial_params_filename != ''}">
-      <xacro:property name="link_inertial_params_file" value="$(find xarm_description)/config/link_inertial/${default_inertial_params_filename}.yaml"/>
+      <xacro:property name="link_inertial_params_file" value="$(find xarm6_description)/config/link_inertial/${default_inertial_params_filename}.yaml"/>
     </xacro:unless>
     <xacro:if value="${use_xacro_load_yaml}">

File: src/robot_descriptions/xarm6_description/urdf/lite6/lite6_robot_macro.xacro (robot description, xacro)
@@ -18,9 +18,9 @@
     <!-- include lite6 relative macros: -->
     <xacro:if value="${is_ros2}">
-      <xacro:include filename="$(find xarm_description)/urdf/lite6/lite6.ros2_control.xacro" />
+      <xacro:include filename="$(find xarm6_description)/urdf/lite6/lite6.ros2_control.xacro" />
     </xacro:if>
-    <xacro:include filename="$(find xarm_description)/urdf/lite6/lite6.urdf.xacro" />
-    <xacro:include filename="$(find xarm_description)/urdf/lite6/lite6.transmission.xacro" />
-    <xacro:include filename="$(find xarm_description)/urdf/lite6/lite6.gazebo.xacro" />
+    <xacro:include filename="$(find xarm6_description)/urdf/lite6/lite6.urdf.xacro" />
+    <xacro:include filename="$(find xarm6_description)/urdf/lite6/lite6.transmission.xacro" />
+    <xacro:include filename="$(find xarm6_description)/urdf/lite6/lite6.gazebo.xacro" />
     <xacro:if value="${limited}">
       <xacro:if value="${is_ros2}">

File: src/robot_descriptions/xarm6_description/urdf/uf850/uf850.urdf.xacro (robot description, xacro)
@@ -14,8 +14,8 @@
     <xacro:property name="default_inertial_params_filename" value="xarm6_type12_HT_LDBR2"/>
     <xacro:if value="${inertial_params_filename != ''}">
-      <xacro:property name="link_inertial_params_file" value="$(find xarm_description)/config/link_inertial/${inertial_params_filename}.yaml"/>
+      <xacro:property name="link_inertial_params_file" value="$(find xarm6_description)/config/link_inertial/${inertial_params_filename}.yaml"/>
     </xacro:if>
     <xacro:unless value="${inertial_params_filename != ''}">
-      <xacro:property name="link_inertial_params_file" value="$(find xarm_description)/config/link_inertial/${default_inertial_params_filename}.yaml"/>
+      <xacro:property name="link_inertial_params_file" value="$(find xarm6_description)/config/link_inertial/${default_inertial_params_filename}.yaml"/>
     </xacro:unless>
     <xacro:if value="${use_xacro_load_yaml}">

File: src/robot_descriptions/xarm6_description/urdf/uf850/uf850_robot_macro.xacro (robot description, xacro)
@@ -20,9 +20,9 @@
     <!-- include uf850 relative macros: -->
     <xacro:if value="${is_ros2}">
-      <xacro:include filename="$(find xarm_description)/urdf/uf850/uf850.ros2_control.xacro" />
+      <xacro:include filename="$(find xarm6_description)/urdf/uf850/uf850.ros2_control.xacro" />
     </xacro:if>
-    <xacro:include filename="$(find xarm_description)/urdf/uf850/uf850.urdf.xacro" />
-    <xacro:include filename="$(find xarm_description)/urdf/uf850/uf850.transmission.xacro" />
-    <xacro:include filename="$(find xarm_description)/urdf/uf850/uf850.gazebo.xacro" />
+    <xacro:include filename="$(find xarm6_description)/urdf/uf850/uf850.urdf.xacro" />
+    <xacro:include filename="$(find xarm6_description)/urdf/uf850/uf850.transmission.xacro" />
+    <xacro:include filename="$(find xarm6_description)/urdf/uf850/uf850.gazebo.xacro" />
     <xacro:if value="${limited}">
       <xacro:if value="${is_ros2}">

File: src/robot_descriptions/xarm6_description/urdf/vacuum_gripper/vacuum_gripper.urdf.xacro (robot description, xacro)
@@ -4,5 +4,5 @@
   <xacro:arg name="prefix" default=""/>
   <xacro:arg name="mesh_suffix" default="stl"/>
-  <xacro:include filename="$(find xarm_description)/urdf/vacuum_gripper/vacuum_gripper_macro.xacro" />
+  <xacro:include filename="$(find xarm6_description)/urdf/vacuum_gripper/vacuum_gripper_macro.xacro" />
   <xacro:vacuum_gripper_device robot_type="$(arg robot_type)" prefix="$(arg prefix)" mesh_suffix="$(arg mesh_suffix)" />
 </robot>

File: src/robot_descriptions/xarm6_description/urdf/vacuum_gripper/vacuum_gripper_macro.xacro (robot description, xacro)
@@ -3,20 +3,20 @@
   <xacro:macro name="vacuum_gripper_device" params="prefix:='' robot_type:='xarm' mesh_suffix:='stl' ">
     <!-- Load Common Material -->
-    <xacro:include filename="$(find xarm_description)/urdf/_private_macro.xacro" />
+    <xacro:include filename="$(find xarm6_description)/urdf/_private_macro.xacro" />
     <xacro:device_macro_begin />
     <!-- Load Common Material -->
-    <xacro:include filename="$(find xarm_description)/urdf/common/common.material.xacro" />
+    <xacro:include filename="$(find xarm6_description)/urdf/common/common.material.xacro" />
     <xacro:common_material prefix="${prefix}"/>
-    <xacro:property name="mesh_path" value="package://xarm_description/meshes" scope="parent"/>
+    <xacro:property name="mesh_path" value="package://xarm6_description/meshes" scope="parent"/>
     <!-- include common.link.xacro -->
-    <xacro:include filename="$(find xarm_description)/urdf/common/common.link.xacro" />
+    <xacro:include filename="$(find xarm6_description)/urdf/common/common.link.xacro" />
     <xacro:if value="${robot_type == 'lite'}">
       <!-- Load Lite Gripper Model URDF -->
-      <xacro:include filename="$(find xarm_description)/urdf/vacuum_gripper/lite_vacuum_gripper.urdf.xacro" />
+      <xacro:include filename="$(find xarm6_description)/urdf/vacuum_gripper/lite_vacuum_gripper.urdf.xacro" />
       <xacro:uflite_vacuum_gripper_urdf prefix="${prefix}" />
     </xacro:if>
     <xacro:unless value="${robot_type == 'lite'}">
       <!-- Load XArm Gripper Model URDF -->
-      <xacro:include filename="$(find xarm_description)/urdf/vacuum_gripper/xarm_vacuum_gripper.urdf.xacro" />
+      <xacro:include filename="$(find xarm6_description)/urdf/vacuum_gripper/xarm_vacuum_gripper.urdf.xacro" />
       <xacro:xarm_vacuum_gripper_urdf prefix="${prefix}" />
     </xacro:unless>

File: src/robot_descriptions/xarm6_description/urdf/xarm6/xarm6.urdf.xacro (robot description, xacro)
@@ -23,8 +23,8 @@
     <xacro:property name="default_inertial_params_filename" value="xarm6_type6_HT_BR2"/>
     <xacro:if value="${inertial_params_filename != ''}">
-      <xacro:property name="link_inertial_params_file" value="$(find xarm_description)/config/link_inertial/${inertial_params_filename}.yaml"/>
+      <xacro:property name="link_inertial_params_file" value="$(find xarm6_description)/config/link_inertial/${inertial_params_filename}.yaml"/>
     </xacro:if>
     <xacro:unless value="${inertial_params_filename != ''}">
-      <xacro:property name="link_inertial_params_file" value="$(find xarm_description)/config/link_inertial/${default_inertial_params_filename}.yaml"/>
+      <xacro:property name="link_inertial_params_file" value="$(find xarm6_description)/config/link_inertial/${default_inertial_params_filename}.yaml"/>
     </xacro:unless>
     <xacro:if value="${use_xacro_load_yaml}">

File: src/robot_descriptions/xarm6_description/urdf/xarm6/xarm6_robot_macro.xacro (robot description, xacro)
@@ -20,9 +20,9 @@
     <!-- include xarm6 relative macros: -->
     <xacro:if value="${is_ros2}">
-      <xacro:include filename="$(find xarm_description)/urdf/xarm6/xarm6.ros2_control.xacro" />
+      <xacro:include filename="$(find xarm6_description)/urdf/xarm6/xarm6.ros2_control.xacro" />
     </xacro:if>
-    <xacro:include filename="$(find xarm_description)/urdf/xarm6/xarm6.urdf.xacro" />
-    <xacro:include filename="$(find xarm_description)/urdf/xarm6/xarm6.transmission.xacro" />
-    <xacro:include filename="$(find xarm_description)/urdf/xarm6/xarm6.gazebo.xacro" />
+    <xacro:include filename="$(find xarm6_description)/urdf/xarm6/xarm6.urdf.xacro" />
+    <xacro:include filename="$(find xarm6_description)/urdf/xarm6/xarm6.transmission.xacro" />
+    <xacro:include filename="$(find xarm6_description)/urdf/xarm6/xarm6.gazebo.xacro" />
     <xacro:if value="${limited}">
       <xacro:if value="${is_ros2}">

File: src/robot_descriptions/xarm6_description/urdf/xarm_device.urdf.xacro (robot description, xacro)
@@ -40,5 +40,5 @@
   <xacro:arg name="kinematics_suffix" default=""/>
   <!-- load xarm device -->
-  <xacro:include filename="$(find xarm_description)/urdf/xarm_device_macro.xacro" />
+  <xacro:include filename="$(find xarm6_description)/urdf/xarm_device_macro.xacro" />
   <xacro:xarm_device prefix="$(arg prefix)" hw_ns="$(arg hw_ns)" limited="$(arg limited)"
     effort_control="$(arg effort_control)" velocity_control="$(arg velocity_control)"
