Commit message: replacing

File: src/robot_descriptions/xarm6_description/urdf/xarm_device_macro.xacro (robot description, xacro)
@@ -45,8 +45,8 @@
     >
     <!-- Load Common Material -->
-    <xacro:include filename="$(find xarm_description)/urdf/_private_macro.xacro" />
+    <xacro:include filename="$(find xarm6_description)/urdf/_private_macro.xacro" />
     <xacro:device_macro_begin />
     <!-- Load Common Material -->
-    <xacro:include filename="$(find xarm_description)/urdf/common/common.material.xacro" />
+    <xacro:include filename="$(find xarm6_description)/urdf/common/common.material.xacro" />
     <xacro:common_material prefix="${prefix}"/>
     <!-- Specify Mesh file path -->
@@ -54,11 +54,11 @@
     <xacro:if value="${ros2_control_plugin == 'gazebo_ros2_control/GazeboSystem' or ros2_control_plugin == 'ign_ros2_control/IgnitionSystem'}">
       <!-- gazebo use -->
-      <xacro:property name="mesh_path" value="file://$(find xarm_description)/meshes" scope="parent"/>
+      <xacro:property name="mesh_path" value="file://$(find xarm6_description)/meshes" scope="parent"/>
     </xacro:if>
     <xacro:unless value="${ros2_control_plugin == 'gazebo_ros2_control/GazeboSystem' or ros2_control_plugin == 'ign_ros2_control/IgnitionSystem'}">
-      <xacro:property name="mesh_path" value="package://xarm_description/meshes" scope="parent"/>
+      <xacro:property name="mesh_path" value="package://xarm6_description/meshes" scope="parent"/>
     </xacro:unless>
     <!-- include common.link.xacro -->
-    <xacro:include filename="$(find xarm_description)/urdf/common/common.link.xacro" />
+    <xacro:include filename="$(find xarm6_description)/urdf/common/common.link.xacro" />
     <xacro:parse_link_inertial_filename dof="${dof}" robot_type="${robot_type}" robot_sn="${robot_sn}" model1300="${model1300}" />
     <xacro:property name="inertial_params_filename" value="${scope_parent_inertial_params_filename}"/>
@@ -91,12 +91,12 @@
     </xacro:unless>
     <xacro:if value="${kinematics_suffix != ''}">
-      <xacro:property name="kinematics_params_filename" value="$(find xarm_description)/config/kinematics/user/${robot_name}_kinematics_${kinematics_suffix}.yaml"/>
+      <xacro:property name="kinematics_params_filename" value="$(find xarm6_description)/config/kinematics/user/${robot_name}_kinematics_${kinematics_suffix}.yaml"/>
     </xacro:if>
     <xacro:unless value="${kinematics_suffix != ''}">
-      <xacro:property name="kinematics_params_filename" value="$(find xarm_description)/config/kinematics/default/${robot_name}_default_kinematics.yaml"/>
+      <xacro:property name="kinematics_params_filename" value="$(find xarm6_description)/config/kinematics/default/${robot_name}_default_kinematics.yaml"/>
     </xacro:unless>
     <xacro:if value="${dof == 5}">
       <!-- Load XArm5 Robot Model URDF -->
-      <xacro:include filename="$(find xarm_description)/urdf/xarm5/xarm5_robot_macro.xacro" />
+      <xacro:include filename="$(find xarm6_description)/urdf/xarm5/xarm5_robot_macro.xacro" />
       <xacro:xarm5_robot prefix="${prefix}" hw_ns="${hw_ns}" limited="${limited}"
         velocity_control="${velocity_control}"
@@ -116,5 +116,5 @@
       <xacro:if value="${robot_type == 'uf850'}">
         <!-- Load UFACTORY 850 Robot Model URDF -->
-        <xacro:include filename="$(find xarm_description)/urdf/uf850/uf850_robot_macro.xacro" />
+        <xacro:include filename="$(find xarm6_description)/urdf/uf850/uf850_robot_macro.xacro" />
         <xacro:uf850_robot prefix="${prefix}" hw_ns="${hw_ns}" limited="${limited}"
           velocity_control="${velocity_control}"
@@ -133,5 +133,5 @@
       <xacro:if value="${robot_type == 'lite'}">
         <!-- Load Lite6 Robot Model URDF -->
-        <xacro:include filename="$(find xarm_description)/urdf/lite6/lite6_robot_macro.xacro" />
+        <xacro:include filename="$(find xarm6_description)/urdf/lite6/lite6_robot_macro.xacro" />
         <xacro:lite6_robot prefix="${prefix}" hw_ns="${hw_ns}" limited="${limited}"
           velocity_control="${velocity_control}"
@@ -148,5 +148,5 @@
       <xacro:unless value="${robot_type == 'lite' or robot_type == 'uf850'}">
         <!-- Load XArm6 Robot Model URDF -->
-        <xacro:include filename="$(find xarm_description)/urdf/xarm6/xarm6_robot_macro.xacro" />
+        <xacro:include filename="$(find xarm6_description)/urdf/xarm6/xarm6_robot_macro.xacro" />
         <xacro:xarm6_robot prefix="${prefix}" hw_ns="${hw_ns}" limited="${limited}"
           velocity_control="${velocity_control}"
@@ -167,5 +167,5 @@
       <xacro:if value="${robot_type == 'xarm7_mirror'}">
         <!-- Load xArm7 Mirror Robot Model URDF -->
-        <xacro:include filename="$(find xarm_description)/urdf/xarm7_mirror/xarm7_mirror_robot_macro.xacro" />
+        <xacro:include filename="$(find xarm6_description)/urdf/xarm7_mirror/xarm7_mirror_robot_macro.xacro" />
         <xacro:xarm7_mirror_robot prefix="${prefix}" hw_ns="${hw_ns}" limited="${limited}"
           velocity_control="${velocity_control}"
@@ -184,5 +184,5 @@
       <xacro:unless value="${robot_type == 'xarm7_mirror'}">
         <!-- Load XArm7 Robot Model URDF -->
-        <xacro:include filename="$(find xarm_description)/urdf/xarm7/xarm7_robot_macro.xacro" />
+        <xacro:include filename="$(find xarm6_description)/urdf/xarm7/xarm7_robot_macro.xacro" />
         <xacro:xarm7_robot prefix="${prefix}" hw_ns="${hw_ns}" limited="${limited}"
           velocity_control="${velocity_control}"
@@ -202,8 +202,8 @@
     <xacro:if value="${add_realsense_d435i}">
       <!-- (xarm) Load RealSense D435i URDF -->
-      <xacro:include filename="$(find xarm_description)/urdf/camera/realsense_d435i.urdf.xacro" />
+      <xacro:include filename="$(find xarm6_description)/urdf/camera/realsense_d435i.urdf.xacro" />
       <xacro:d435i_urdf prefix="${prefix}" add_d435i_links="${add_d435i_links}" />
       <xacro:if value="${add_d435i_links}">
-        <xacro:include filename="$(find xarm_description)/urdf/camera/realsense.gazebo.xacro" />
+        <xacro:include filename="$(find xarm6_description)/urdf/camera/realsense.gazebo.xacro" />
         <xacro:realsense_gazebo prefix="${prefix}" />
       </xacro:if>
@@ -220,10 +220,10 @@
       <xacro:if value="${robot_type == 'lite'}">
         <!-- Load Lite Gripper Model URDF -->
-        <xacro:include filename="$(find xarm_description)/urdf/gripper/lite_gripper.urdf.xacro" />
+        <xacro:include filename="$(find xarm6_description)/urdf/gripper/lite_gripper.urdf.xacro" />
         <xacro:uflite_gripper_urdf prefix="${prefix}" attach_to="${prefix}link_eef" />
       </xacro:if>
       <xacro:unless value="${robot_type == 'lite'}">
         <!-- Load XArm Gripper Model URDF -->
-        <xacro:include filename="$(find xarm_description)/urdf/gripper/xarm_gripper_macro.xacro" />
+        <xacro:include filename="$(find xarm6_description)/urdf/gripper/xarm_gripper_macro.xacro" />
         <xacro:xarm_gripper_macro prefix="${prefix}" attach_to="${prefix}link_eef"
           ros2_control_plugin="${ros2_control_plugin}" dof="${dof}" hard_interface="${hard_interface}" />
@@ -233,5 +233,5 @@
       <xacro:unless value="${robot_type == 'lite'}">
         <!-- Load BIO Gripper Model URDF -->
-        <xacro:include filename="$(find xarm_description)/urdf/gripper/bio_gripper_macro.xacro" />
+        <xacro:include filename="$(find xarm6_description)/urdf/gripper/bio_gripper_macro.xacro" />
         <xacro:bio_gripper_macro prefix="${prefix}" attach_to="${prefix}link_eef"
           ros2_control_plugin="${ros2_control_plugin}" dof="${dof}" hard_interface="${hard_interface}" />
@@ -241,10 +241,10 @@
       <xacro:if value="${robot_type == 'lite'}">
         <!-- Load Lite Vacuum Gripper Model URDF -->
-        <xacro:include filename="$(find xarm_description)/urdf/vacuum_gripper/lite_vacuum_gripper.urdf.xacro" />
+        <xacro:include filename="$(find xarm6_description)/urdf/vacuum_gripper/lite_vacuum_gripper.urdf.xacro" />
         <xacro:uflite_vacuum_gripper_urdf prefix="${prefix}" attach_to="${prefix}link_eef" />
       </xacro:if>
       <xacro:unless value="${robot_type == 'lite'}">
         <!-- Load XArm Vacuum Gripper Model URDF -->
-        <xacro:include filename="$(find xarm_description)/urdf/vacuum_gripper/xarm_vacuum_gripper.urdf.xacro" />
+        <xacro:include filename="$(find xarm6_description)/urdf/vacuum_gripper/xarm_vacuum_gripper.urdf.xacro" />
         <xacro:xarm_vacuum_gripper_urdf prefix="${prefix}" attach_to="${prefix}link_eef" />
       </xacro:unless>
@@ -252,5 +252,5 @@
     <xacro:if value="${not add_gripper and not add_vacuum_gripper and add_other_geometry}">
       <!-- Load Other Model URDF -->
-      <xacro:include filename="$(find xarm_description)/urdf/other/other_geometry.urdf.xacro" />
+      <xacro:include filename="$(find xarm6_description)/urdf/other/other_geometry.urdf.xacro" />
       <xacro:other_geometry prefix="${prefix}" attach_to="${prefix}link_eef"
         geometry_type="${geometry_type}" geometry_mass="${geometry_mass}"
@@ -264,5 +264,5 @@
     <!-- gazebo_plugin -->
     <xacro:if value="${load_gazebo_plugin}">
-      <xacro:include filename="$(find xarm_description)/urdf/common/common.gazebo.xacro" />
+      <xacro:include filename="$(find xarm6_description)/urdf/common/common.gazebo.xacro" />
       <xacro:if value="${is_ros2}">
         <xacro:if value="${robot_type == 'uf850' or robot_type == 'xarm7_mirror'}">
@@ -287,5 +287,5 @@
     </xacro:if>
     <xacro:if value="${use_gazebo_camera}">
-      <xacro:include filename="$(find xarm_description)/urdf/camera/camera.gazebo.xacro" />
+      <xacro:include filename="$(find xarm6_description)/urdf/camera/camera.gazebo.xacro" />
       <xacro:camera_gazebo prefix="${prefix}" />
     </xacro:if>
