Commit message: rviz

File: src/robot_descriptions/xarm6_description/urdf/xarm_device_macro.xacro (robot description, xacro)
@@ -217,4 +217,26 @@
       <child link="${prefix}link_eef" />
     </joint>
+  <!-- Define the position and orientation of the camera in the environment -->
+  <link name="${prefix}realsense_camera_link">
+    <origin xyz="1 2 1.5" rpy="0.785 0 1.57" />
+  </link>
+  <joint name="${prefix}realsense_camera_joint" type="fixed">
+    <origin xyz="0 0 0" rpy="0 0 0" />
+    <parent link="world"/>
+    <child link="${prefix}realsense_camera_link" />
+  </joint>
+  <!-- Attach the RealSense camera to the newly defined link -->
+  <xacro:d435i_urdf prefix="${prefix}realsense_camera_" add_d435i_links="${add_d435i_links}" />
+  <xacro:if value="${add_d435i_links}">
+    <xacro:include filename="$(find xarm6_description)/urdf/camera/realsense.gazebo.xacro" />
+    <xacro:realsense_gazebo prefix="${prefix}realsense_camera_" />
+  </xacro:if>
+</xacro:if>
+<!-- Optional: Any additional environment or robot links can be defined here -->
+<joint name="${prefix}joint_eef" type="fixed">
+  <origin xyz="0 0 0" rpy="0 0 0" />
+  <parent link="${prefix}link${dof}" />
+  <child link="${prefix}link_eef" />
+</joint>
     <xacro:if value="${add_gripper}">
       <xacro:if value="${robot_type == 'lite'}">

Commit message: Rviz Working with camera

File: src/robot_descriptions/xarm6_description/urdf/xarm_device_macro.xacro (robot description, xacro)
@@ -45,8 +45,8 @@
     >
     <!-- Load Common Material -->
-    <xacro:include filename="$(find xarm6_description)/urdf/_private_macro.xacro" />
+    <xacro:include filename="$(find xarm_description)/urdf/_private_macro.xacro" />
     <xacro:device_macro_begin />
     <!-- Load Common Material -->
-    <xacro:include filename="$(find xarm6_description)/urdf/common/common.material.xacro" />
+    <xacro:include filename="$(find xarm_description)/urdf/common/common.material.xacro" />
     <xacro:common_material prefix="${prefix}"/>
     <!-- Specify Mesh file path -->
@@ -54,11 +54,11 @@
     <xacro:if value="${ros2_control_plugin == 'gazebo_ros2_control/GazeboSystem' or ros2_control_plugin == 'ign_ros2_control/IgnitionSystem'}">
       <!-- gazebo use -->
-      <xacro:property name="mesh_path" value="file://$(find xarm6_description)/meshes" scope="parent"/>
+      <xacro:property name="mesh_path" value="file://$(find xarm_description)/meshes" scope="parent"/>
     </xacro:if>
     <xacro:unless value="${ros2_control_plugin == 'gazebo_ros2_control/GazeboSystem' or ros2_control_plugin == 'ign_ros2_control/IgnitionSystem'}">
-      <xacro:property name="mesh_path" value="package://xarm6_description/meshes" scope="parent"/>
+      <xacro:property name="mesh_path" value="package://xarm_description/meshes" scope="parent"/>
     </xacro:unless>
     <!-- include common.link.xacro -->
-    <xacro:include filename="$(find xarm6_description)/urdf/common/common.link.xacro" />
+    <xacro:include filename="$(find xarm_description)/urdf/common/common.link.xacro" />
     <xacro:parse_link_inertial_filename dof="${dof}" robot_type="${robot_type}" robot_sn="${robot_sn}" model1300="${model1300}" />
     <xacro:property name="inertial_params_filename" value="${scope_parent_inertial_params_filename}"/>
@@ -91,12 +91,12 @@
     </xacro:unless>
     <xacro:if value="${kinematics_suffix != ''}">
-      <xacro:property name="kinematics_params_filename" value="$(find xarm6_description)/config/kinematics/user/${robot_name}_kinematics_${kinematics_suffix}.yaml"/>
+      <xacro:property name="kinematics_params_filename" value="$(find xarm_description)/config/kinematics/user/${robot_name}_kinematics_${kinematics_suffix}.yaml"/>
     </xacro:if>
     <xacro:unless value="${kinematics_suffix != ''}">
-      <xacro:property name="kinematics_params_filename" value="$(find xarm6_description)/config/kinematics/default/${robot_name}_default_kinematics.yaml"/>
+      <xacro:property name="kinematics_params_filename" value="$(find xarm_description)/config/kinematics/default/${robot_name}_default_kinematics.yaml"/>
     </xacro:unless>
     <xacro:if value="${dof == 5}">
       <!-- Load XArm5 Robot Model URDF -->
-      <xacro:include filename="$(find xarm6_description)/urdf/xarm5/xarm5_robot_macro.xacro" />
+      <xacro:include filename="$(find xarm_description)/urdf/xarm5/xarm5_robot_macro.xacro" />
       <xacro:xarm5_robot prefix="${prefix}" hw_ns="${hw_ns}" limited="${limited}"
         velocity_control="${velocity_control}"
@@ -116,5 +116,5 @@
       <xacro:if value="${robot_type == 'uf850'}">
         <!-- Load UFACTORY 850 Robot Model URDF -->
-        <xacro:include filename="$(find xarm6_description)/urdf/uf850/uf850_robot_macro.xacro" />
+        <xacro:include filename="$(find xarm_description)/urdf/uf850/uf850_robot_macro.xacro" />
         <xacro:uf850_robot prefix="${prefix}" hw_ns="${hw_ns}" limited="${limited}"
           velocity_control="${velocity_control}"
@@ -133,5 +133,5 @@
       <xacro:if value="${robot_type == 'lite'}">
         <!-- Load Lite6 Robot Model URDF -->
-        <xacro:include filename="$(find xarm6_description)/urdf/lite6/lite6_robot_macro.xacro" />
+        <xacro:include filename="$(find xarm_description)/urdf/lite6/lite6_robot_macro.xacro" />
         <xacro:lite6_robot prefix="${prefix}" hw_ns="${hw_ns}" limited="${limited}"
           velocity_control="${velocity_control}"
@@ -148,5 +148,5 @@
       <xacro:unless value="${robot_type == 'lite' or robot_type == 'uf850'}">
         <!-- Load XArm6 Robot Model URDF -->
-        <xacro:include filename="$(find xarm6_description)/urdf/xarm6/xarm6_robot_macro.xacro" />
+        <xacro:include filename="$(find xarm_description)/urdf/xarm6/xarm6_robot_macro.xacro" />
         <xacro:xarm6_robot prefix="${prefix}" hw_ns="${hw_ns}" limited="${limited}"
           velocity_control="${velocity_control}"
@@ -167,5 +167,5 @@
       <xacro:if value="${robot_type == 'xarm7_mirror'}">
         <!-- Load xArm7 Mirror Robot Model URDF -->
-        <xacro:include filename="$(find xarm6_description)/urdf/xarm7_mirror/xarm7_mirror_robot_macro.xacro" />
+        <xacro:include filename="$(find xarm_description)/urdf/xarm7_mirror/xarm7_mirror_robot_macro.xacro" />
         <xacro:xarm7_mirror_robot prefix="${prefix}" hw_ns="${hw_ns}" limited="${limited}"
           velocity_control="${velocity_control}"
@@ -184,5 +184,5 @@
       <xacro:unless value="${robot_type == 'xarm7_mirror'}">
         <!-- Load XArm7 Robot Model URDF -->
-        <xacro:include filename="$(find xarm6_description)/urdf/xarm7/xarm7_robot_macro.xacro" />
+        <xacro:include filename="$(find xarm_description)/urdf/xarm7/xarm7_robot_macro.xacro" />
         <xacro:xarm7_robot prefix="${prefix}" hw_ns="${hw_ns}" limited="${limited}"
           velocity_control="${velocity_control}"
@@ -202,8 +202,8 @@
     <xacro:if value="${add_realsense_d435i}">
       <!-- (xarm) Load RealSense D435i URDF -->
-      <xacro:include filename="$(find xarm6_description)/urdf/camera/realsense_d435i.urdf.xacro" />
+      <xacro:include filename="$(find xarm_description)/urdf/camera/realsense_d435i.urdf.xacro" />
       <xacro:d435i_urdf prefix="${prefix}" add_d435i_links="${add_d435i_links}" />
       <xacro:if value="${add_d435i_links}">
-        <xacro:include filename="$(find xarm6_description)/urdf/camera/realsense.gazebo.xacro" />
+        <xacro:include filename="$(find xarm_description)/urdf/camera/realsense.gazebo.xacro" />
         <xacro:realsense_gazebo prefix="${prefix}" />
       </xacro:if>
@@ -217,35 +217,13 @@
       <child link="${prefix}link_eef" />
     </joint>
-  <!-- Define the position and orientation of the camera in the environment -->
-  <link name="${prefix}realsense_camera_link">
-    <origin xyz="1 2 1.5" rpy="0.785 0 1.57" />
-  </link>
-  <joint name="${prefix}realsense_camera_joint" type="fixed">
-    <origin xyz="0 0 0" rpy="0 0 0" />
-    <parent link="world"/>
-    <child link="${prefix}realsense_camera_link" />
-  </joint>
-  <!-- Attach the RealSense camera to the newly defined link -->
-  <xacro:d435i_urdf prefix="${prefix}realsense_camera_" add_d435i_links="${add_d435i_links}" />
-  <xacro:if value="${add_d435i_links}">
-    <xacro:include filename="$(find xarm6_description)/urdf/camera/realsense.gazebo.xacro" />
-    <xacro:realsense_gazebo prefix="${prefix}realsense_camera_" />
-  </xacro:if>
-</xacro:if>
-<!-- Optional: Any additional environment or robot links can be defined here -->
-<joint name="${prefix}joint_eef" type="fixed">
-  <origin xyz="0 0 0" rpy="0 0 0" />
-  <parent link="${prefix}link${dof}" />
-  <child link="${prefix}link_eef" />
-</joint>
     <xacro:if value="${add_gripper}">
       <xacro:if value="${robot_type == 'lite'}">
         <!-- Load Lite Gripper Model URDF -->
-        <xacro:include filename="$(find xarm6_description)/urdf/gripper/lite_gripper.urdf.xacro" />
+        <xacro:include filename="$(find xarm_description)/urdf/gripper/lite_gripper.urdf.xacro" />
         <xacro:uflite_gripper_urdf prefix="${prefix}" attach_to="${prefix}link_eef" />
       </xacro:if>
       <xacro:unless value="${robot_type == 'lite'}">
         <!-- Load XArm Gripper Model URDF -->
-        <xacro:include filename="$(find xarm6_description)/urdf/gripper/xarm_gripper_macro.xacro" />
+        <xacro:include filename="$(find xarm_description)/urdf/gripper/xarm_gripper_macro.xacro" />
         <xacro:xarm_gripper_macro prefix="${prefix}" attach_to="${prefix}link_eef"
           ros2_control_plugin="${ros2_control_plugin}" dof="${dof}" hard_interface="${hard_interface}" />
@@ -255,5 +233,5 @@
       <xacro:unless value="${robot_type == 'lite'}">
         <!-- Load BIO Gripper Model URDF -->
-        <xacro:include filename="$(find xarm6_description)/urdf/gripper/bio_gripper_macro.xacro" />
+        <xacro:include filename="$(find xarm_description)/urdf/gripper/bio_gripper_macro.xacro" />
         <xacro:bio_gripper_macro prefix="${prefix}" attach_to="${prefix}link_eef"
           ros2_control_plugin="${ros2_control_plugin}" dof="${dof}" hard_interface="${hard_interface}" />
@@ -263,10 +241,10 @@
       <xacro:if value="${robot_type == 'lite'}">
         <!-- Load Lite Vacuum Gripper Model URDF -->
-        <xacro:include filename="$(find xarm6_description)/urdf/vacuum_gripper/lite_vacuum_gripper.urdf.xacro" />
+        <xacro:include filename="$(find xarm_description)/urdf/vacuum_gripper/lite_vacuum_gripper.urdf.xacro" />
         <xacro:uflite_vacuum_gripper_urdf prefix="${prefix}" attach_to="${prefix}link_eef" />
       </xacro:if>
       <xacro:unless value="${robot_type == 'lite'}">
         <!-- Load XArm Vacuum Gripper Model URDF -->
-        <xacro:include filename="$(find xarm6_description)/urdf/vacuum_gripper/xarm_vacuum_gripper.urdf.xacro" />
+        <xacro:include filename="$(find xarm_description)/urdf/vacuum_gripper/xarm_vacuum_gripper.urdf.xacro" />
         <xacro:xarm_vacuum_gripper_urdf prefix="${prefix}" attach_to="${prefix}link_eef" />
       </xacro:unless>
@@ -274,5 +252,5 @@
     <xacro:if value="${not add_gripper and not add_vacuum_gripper and add_other_geometry}">
       <!-- Load Other Model URDF -->
-      <xacro:include filename="$(find xarm6_description)/urdf/other/other_geometry.urdf.xacro" />
+      <xacro:include filename="$(find xarm_description)/urdf/other/other_geometry.urdf.xacro" />
       <xacro:other_geometry prefix="${prefix}" attach_to="${prefix}link_eef"
         geometry_type="${geometry_type}" geometry_mass="${geometry_mass}"
@@ -286,5 +264,5 @@
     <!-- gazebo_plugin -->
     <xacro:if value="${load_gazebo_plugin}">
-      <xacro:include filename="$(find xarm6_description)/urdf/common/common.gazebo.xacro" />
+      <xacro:include filename="$(find xarm_description)/urdf/common/common.gazebo.xacro" />
       <xacro:if value="${is_ros2}">
         <xacro:if value="${robot_type == 'uf850' or robot_type == 'xarm7_mirror'}">
@@ -309,5 +287,5 @@
     </xacro:if>
     <xacro:if value="${use_gazebo_camera}">
-      <xacro:include filename="$(find xarm6_description)/urdf/camera/camera.gazebo.xacro" />
+      <xacro:include filename="$(find xarm_description)/urdf/camera/camera.gazebo.xacro" />
       <xacro:camera_gazebo prefix="${prefix}" />
     </xacro:if>

Commit message: cleaning xacro files

File: src/robot_descriptions/xarm6_description/urdf/xarm_device_macro.xacro (robot description, xacro)
@@ -96,54 +96,5 @@
       <xacro:property name="kinematics_params_filename" value="$(find xarm6_description)/config/kinematics/default/${robot_name}_default_kinematics.yaml"/>
     </xacro:unless>
-    <xacro:if value="${dof == 5}">
-      <!-- Load XArm5 Robot Model URDF -->
-      <xacro:include filename="$(find xarm6_description)/urdf/xarm5/xarm5_robot_macro.xacro" />
-      <xacro:xarm5_robot prefix="${prefix}" hw_ns="${hw_ns}" limited="${limited}"
-        velocity_control="${velocity_control}"
-        ros2_control_plugin="${ros2_control_plugin}"
-        add_gripper="${add_gripper}"
-        add_bio_gripper="${add_bio_gripper}"
-        robot_ip="${robot_ip}"
-        report_type="${report_type}"
-        baud_checkset="${baud_checkset}"
-        default_gripper_baud="${default_gripper_baud}"
-        model1300="${new_model1300}"
-        inertial_params_filename="${inertial_params_filename}"
-        kinematics_params_filename="${kinematics_params_filename}"
-        hard_interface="${hard_interface}" />
-    </xacro:if>
     <xacro:if value="${dof == 6}">
-      <xacro:if value="${robot_type == 'uf850'}">
-        <!-- Load UFACTORY 850 Robot Model URDF -->
-        <xacro:include filename="$(find xarm6_description)/urdf/uf850/uf850_robot_macro.xacro" />
-        <xacro:uf850_robot prefix="${prefix}" hw_ns="${hw_ns}" limited="${limited}"
-          velocity_control="${velocity_control}"
-          ros2_control_plugin="${ros2_control_plugin}"
-          add_gripper="${add_gripper}"
-          add_bio_gripper="${add_bio_gripper}"
-          robot_ip="${robot_ip}"
-          report_type="${report_type}"
-          baud_checkset="${baud_checkset}"
-          default_gripper_baud="${default_gripper_baud}"
-          model1300="${new_model1300}"
-          inertial_params_filename="${inertial_params_filename}"
-          kinematics_params_filename="${kinematics_params_filename}"
-          hard_interface="${hard_interface}" />
-      </xacro:if>
-      <xacro:if value="${robot_type == 'lite'}">
-        <!-- Load Lite6 Robot Model URDF -->
-        <xacro:include filename="$(find xarm6_description)/urdf/lite6/lite6_robot_macro.xacro" />
-        <xacro:lite6_robot prefix="${prefix}" hw_ns="${hw_ns}" limited="${limited}"
-          velocity_control="${velocity_control}"
-          ros2_control_plugin="${ros2_control_plugin}"
-          add_gripper="${add_gripper}"
-          robot_ip="${robot_ip}"
-          report_type="${report_type}"
-          baud_checkset="${baud_checkset}"
-          default_gripper_baud="${default_gripper_baud}"
-          inertial_params_filename="${inertial_params_filename}"
-          kinematics_params_filename="${kinematics_params_filename}"
-          hard_interface="${hard_interface}" />
-      </xacro:if>
       <xacro:unless value="${robot_type == 'lite' or robot_type == 'uf850'}">
         <!-- Load XArm6 Robot Model URDF -->
@@ -164,42 +115,19 @@
       </xacro:unless>
     </xacro:if>
-    <xacro:unless value="${dof == 5 or dof == 6}">
-      <xacro:if value="${robot_type == 'xarm7_mirror'}">
-        <!-- Load xArm7 Mirror Robot Model URDF -->
-        <xacro:include filename="$(find xarm6_description)/urdf/xarm7_mirror/xarm7_mirror_robot_macro.xacro" />
-        <xacro:xarm7_mirror_robot prefix="${prefix}" hw_ns="${hw_ns}" limited="${limited}"
-          velocity_control="${velocity_control}"
-          ros2_control_plugin="${ros2_control_plugin}"
-          add_gripper="${add_gripper}"
-          add_bio_gripper="${add_bio_gripper}"
-          robot_ip="${robot_ip}"
-          report_type="${report_type}"
-          baud_checkset="${baud_checkset}"
-          default_gripper_baud="${default_gripper_baud}"
-          model1300="${new_model1300}"
-          inertial_params_filename="${inertial_params_filename}"
-          kinematics_params_filename="${kinematics_params_filename}"
-          hard_interface="${hard_interface}" />
-      </xacro:if>
-      <xacro:unless value="${robot_type == 'xarm7_mirror'}">
-        <!-- Load XArm7 Robot Model URDF -->
-        <xacro:include filename="$(find xarm6_description)/urdf/xarm7/xarm7_robot_macro.xacro" />
-        <xacro:xarm7_robot prefix="${prefix}" hw_ns="${hw_ns}" limited="${limited}"
-          velocity_control="${velocity_control}"
-          ros2_control_plugin="${ros2_control_plugin}"
-          add_gripper="${add_gripper}"
-          add_bio_gripper="${add_bio_gripper}"
-          robot_ip="${robot_ip}"
-          report_type="${report_type}"
-          baud_checkset="${baud_checkset}"
-          default_gripper_baud="${default_gripper_baud}"
-          model1300="${new_model1300}"
-          inertial_params_filename="${inertial_params_filename}"
-          kinematics_params_filename="${kinematics_params_filename}"
-          hard_interface="${hard_interface}" />
-      </xacro:unless>
-    </xacro:unless>
+    <!-- (xarm) Load RealSense D435i URDF -->
+    <link name="fixed_frame">
+      <visual>
+        <geometry>
+          <box size="0.1 0.1 0.1"/>
+        </geometry>
+        <material name="Black"/>
+      </visual>
+    </link>
+    <joint name="world_to_fixed_frame" type="fixed">
+      <origin xyz="5 5 5" rpy="10 10 10"/>
+      <parent link="${attach_to}"/>
+      <child link="fixed_frame"/>
+    </joint>
     <xacro:if value="${add_realsense_d435i}">
-      <!-- (xarm) Load RealSense D435i URDF -->
       <xacro:include filename="$(find xarm6_description)/urdf/camera/realsense_d435i.urdf.xacro" />
       <xacro:d435i_urdf prefix="${prefix}" add_d435i_links="${add_d435i_links}" />
@@ -210,5 +138,5 @@
     </xacro:if>
     <xacro:unless value="${add_realsense_d435i}">
-      <link name="${prefix}link_eef"/>
+      <link name="fixed_frame"/>
     </xacro:unless>
     <joint name="${prefix}joint_eef" type="fixed">
@@ -218,9 +146,4 @@
     </joint>
     <xacro:if value="${add_gripper}">
-      <xacro:if value="${robot_type == 'lite'}">
-        <!-- Load Lite Gripper Model URDF -->
-        <xacro:include filename="$(find xarm6_description)/urdf/gripper/lite_gripper.urdf.xacro" />
-        <xacro:uflite_gripper_urdf prefix="${prefix}" attach_to="${prefix}link_eef" />
-      </xacro:if>
       <xacro:unless value="${robot_type == 'lite'}">
         <!-- Load XArm Gripper Model URDF -->
@@ -239,9 +162,4 @@
     </xacro:if>
     <xacro:if value="${not add_gripper and not add_bio_gripper and add_vacuum_gripper}">
-      <xacro:if value="${robot_type == 'lite'}">
-        <!-- Load Lite Vacuum Gripper Model URDF -->
-        <xacro:include filename="$(find xarm6_description)/urdf/vacuum_gripper/lite_vacuum_gripper.urdf.xacro" />
-        <xacro:uflite_vacuum_gripper_urdf prefix="${prefix}" attach_to="${prefix}link_eef" />
-      </xacro:if>
       <xacro:unless value="${robot_type == 'lite'}">
         <!-- Load XArm Vacuum Gripper Model URDF -->

Commit message: fixing

File: src/robot_descriptions/xarm6_description/urdf/xarm_device_macro.xacro (robot description, xacro)
@@ -125,5 +125,5 @@
     </link>
     <joint name="world_to_fixed_frame" type="fixed">
-      <origin xyz="5 5 5" rpy="10 10 10"/>
+      <origin xyz="0 0 0" rpy="0 0 0"/>
       <parent link="${attach_to}"/>
       <child link="fixed_frame"/>

Commit message: working camera

File: src/robot_descriptions/xarm6_description/urdf/xarm_device_macro.xacro (robot description, xacro)
@@ -20,5 +20,5 @@
     load_gazebo_plugin:=false
     add_realsense_d435i:=false
-    add_d435i_links:=true
+    add_d435i_links:=false
     use_gazebo_camera:=false
     add_other_geometry:=false
@@ -116,17 +116,4 @@
     </xacro:if>
     <!-- (xarm) Load RealSense D435i URDF -->
-    <link name="fixed_frame">
-      <visual>
-        <geometry>
-          <box size="0.1 0.1 0.1"/>
-        </geometry>
-        <material name="Black"/>
-      </visual>
-    </link>
-    <joint name="world_to_fixed_frame" type="fixed">
-      <origin xyz="0 0 0" rpy="0 0 0"/>
-      <parent link="${attach_to}"/>
-      <child link="fixed_frame"/>
-    </joint>
     <xacro:if value="${add_realsense_d435i}">
       <xacro:include filename="$(find xarm6_description)/urdf/camera/realsense_d435i.urdf.xacro" />

Commit message: Working arm without camera

File: src/robot_descriptions/xarm6_description/urdf/xarm_device_macro.xacro (robot description, xacro)
@@ -125,5 +125,5 @@
     </xacro:if>
     <xacro:unless value="${add_realsense_d435i}">
-      <link name="fixed_frame"/>
+      <link name="${prefix}link_eef"/>
     </xacro:unless>
     <joint name="${prefix}joint_eef" type="fixed">
