Commit message: Working camera

File: src/robot_descriptions/xarm6_description/urdf/camera/camera.gazebo.xacro (robot description, xacro)
@@ -1,4 +1,6 @@
 <?xml version="1.0"?>
 <robot xmlns:xacro="http://ros.org/wiki/xacro">
+  <xacro:property name="M_PI" value="3.1415926535897931" />
+  <xacro:property name="camera_01" value="front_camera" />
   <xacro:macro name="camera_gazebo" params="prefix">
     <link name="${prefix}link_camera">
@@ -25,5 +27,5 @@
     </link>
     <joint name="${prefix}joint_camera" type="fixed">
-      <origin xyz="0.692 0.001 1.17" rpy="0 1.5708 0" />
+      <origin xyz="-1.0 0.5 0.5" rpy="0.0 ${M_PI/10} -${M_PI/7}" />
       <parent link="${prefix}link_base" />
       <child link="${prefix}link_camera" />
@@ -32,19 +34,39 @@
       <material>Gazebo/Black</material>
     </gazebo>
-    <gazebo reference="${prefix}link_camera">
-      <sensor type="camera" name="xarm_camera_node">
-        <!-- <always_on>0</always_on> -->
-        <update_rate>10.0</update_rate>
-        <camera name="head">
-          <!-- <horizontal_fov>1.3962634</horizontal_fov> -->
-          <horizontal_fov>0.9948376567</horizontal_fov>
+   <gazebo reference="${prefix}link_camera">
+      <sensor name="cameradepth" type="depth">
+        <camera name="camera">
+          <horizontal_fov>1.57</horizontal_fov>
           <image>
-            <width>640</width>
-            <height>480</height>
-            <foramt>B8G8R8</foramt>
+            <width>1280</width>
+            <height>720</height>
           </image>
           <clip>
-            <near>0.02</near>
-            <far>300</far>
+            <near>0.1</near>
+            <far>100</far>
+          </clip>
+          <noise>
+            <type>gaussian</type>
+            <mean>0.0</mean>
+            <stddev>0.100</stddev>
+          </noise>
+        </camera>
+        <always_on>1</always_on>
+        <update_rate>30</update_rate>
+        <visualize>0</visualize>
+      </sensor>
+    </gazebo>
+    <gazebo reference="${prefix}link_camera">
+      <sensor name="cameracolor" type="camera">
+        <camera name="camera">
+          <horizontal_fov>1.57</horizontal_fov>
+          <image>
+            <width>1280</width>
+            <height>720</height>
+            <format>RGB_INT8</format>
+          </image>
+          <clip>
+            <near>0.1</near>
+            <far>100</far>
           </clip>
           <noise>
@@ -54,31 +76,77 @@
           </noise>
         </camera>
-        <plugin name="gazebo_camera" filename="libgazebo_ros_camera.so">
-          <xacro:if value="${is_ros2}">
-            <ros>
-              <namespace>/</namespace>
-              <remapping>image_raw:=image_raw</remapping>
-              <remapping>camera_info:=camera_info</remapping>
-            </ros>
-            <camera_name>camera</camera_name>
-            <frame_name>camera_link</frame_name>
-            <hack_baseline>0.07</hack_baseline>
-          </xacro:if>
-          <xacro:unless value="${is_ros2}">
-            <alwaysOn>true</alwaysOn>
-            <updateRate>0.0</updateRate>
-            <cameraName>/camera</cameraName>
-            <imageTopicName>image_raw</imageTopicName>
-            <cameraInfoTopicName>camera_info</cameraInfoTopicName>
-            <frameName>camera_link</frameName>
-            <hackBaseline>0.07</hackBaseline>
-            <distortionK1>0.0</distortionK1>
-            <distortionK2>0.0</distortionK2>
-            <distortionK3>0.0</distortionK3>
-            <distortionT1>0.0</distortionT1>
-            <distortionT2>0.0</distortionT2>
-          </xacro:unless>
-        </plugin>
+        <always_on>1</always_on>
+        <update_rate>30</update_rate>
+        <visualize>1</visualize>
       </sensor>
+    </gazebo>
+    <gazebo reference="${prefix}link_camera">
+      <sensor name="cameraired1" type="camera">
+        <camera name="camera">
+          <horizontal_fov>1.57</horizontal_fov>
+          <image>
+            <width>1280</width>
+            <height>720</height>
+            <format>L_INT8</format>
+          </image>
+          <clip>
+            <near>0.1</near>
+            <far>100</far>
+          </clip>
+          <noise>
+            <type>gaussian</type>
+            <mean>0.0</mean>
+            <stddev>0.05</stddev>
+          </noise>
+        </camera>
+        <always_on>1</always_on>
+        <update_rate>30</update_rate>
+        <visualize>0</visualize>
+      </sensor>
+    </gazebo>
+    <gazebo reference="${prefix}link_camera">
+      <sensor name="cameraired2" type="camera">
+        <camera name="camera">
+          <horizontal_fov>1.57</horizontal_fov>
+          <image>
+            <width>1280</width>
+            <height>720</height>
+            <format>L_INT8</format>
+          </image>
+          <clip>
+            <near>0.1</near>
+            <far>100</far>
+          </clip>
+          <noise>
+            <type>gaussian</type>
+            <mean>0.0</mean>
+            <stddev>0.05</stddev>
+          </noise>
+        </camera>
+        <always_on>1</always_on>
+        <update_rate>30</update_rate>
+        <visualize>0</visualize>
+      </sensor>
+    </gazebo>
+    <gazebo>
+      <plugin name="realsense_gazebo_camera" filename="librealsense_gazebo_plugin.so">
+        <prefix>camera</prefix>
+        <depthUpdateRate>30.0</depthUpdateRate>
+        <colorUpdateRate>30.0</colorUpdateRate>
+        <infraredUpdateRate>30.0</infraredUpdateRate>
+        <depthTopicName>${camera_01}/depth/image_raw</depthTopicName>
+        <depthCameraInfoTopicName>${camera_01}/depth/camera_info</depthCameraInfoTopicName>
+        <colorTopicName>${camera_01}/color/image_raw</colorTopicName>
+        <colorCameraInfoTopicName>${camera_01}/color/camera_info</colorCameraInfoTopicName>
+        <infrared1TopicName>${camera_01}/infra1/image_raw</infrared1TopicName>
+        <infrared1CameraInfoTopicName>${camera_01}/infra1/camera_info</infrared1CameraInfoTopicName>
+        <infrared2TopicName>${camera_01}/infra2/image_raw</infrared2TopicName>
+        <infrared2CameraInfoTopicName>${camera_01}/infra2/camera_info</infrared2CameraInfoTopicName>
+        <rangeMinDepth>0.3</rangeMinDepth>
+        <rangeMaxDepth>3.0</rangeMaxDepth>
+        <pointCloud>true</pointCloud>
+        <pointCloudTopicName>${camera_01}/depth/color/points</pointCloudTopicName>
+        <pointCloudCutoff>0.3</pointCloudCutoff>
+      </plugin>
     </gazebo>
   </xacro:macro>

Commit message: Working point cloud

File: src/robot_descriptions/xarm6_description/urdf/camera/camera.gazebo.xacro (robot description, xacro)
@@ -2,7 +2,7 @@
 <robot xmlns:xacro="http://ros.org/wiki/xacro">
   <xacro:property name="M_PI" value="3.1415926535897931" />
-  <xacro:property name="camera_01" value="front_camera" />
+  <xacro:property name="camera_01" value="camera_front" />
   <xacro:macro name="camera_gazebo" params="prefix">
-    <link name="${prefix}link_camera">
+    <link name="${camera_01}_link_camera">
       <inertial>
         <origin xyz="0 0 0" rpy="0 0 0" />
@@ -26,13 +26,61 @@
       </collision>
     </link>
-    <joint name="${prefix}joint_camera" type="fixed">
+    <link name="${camera_01}_camera_depth_frame"></link>
+    <link name="${camera_01}_camera_depth_optical_frame"></link>
+    <link name="${camera_01}_camera_color_frame"></link>
+    <link name="${camera_01}_camera_color_optical_frame"></link>
+    <link name="${camera_01}_camera_left_ir_frame"></link>
+    <link name="${camera_01}_camera_left_ir_optical_frame"></link>
+    <link name="${camera_01}_camera_right_ir_frame"></link>
+    <link name="${camera_01}_camera_right_ir_optical_frame"></link>
+    <joint name="${camera_01}_joint_camera" type="fixed">
       <origin xyz="-1.0 0.5 0.5" rpy="0.0 ${M_PI/10} -${M_PI/7}" />
       <parent link="${prefix}link_base" />
-      <child link="${prefix}link_camera" />
-    </joint>
-    <gazebo reference="${prefix}link_camera">
+      <child link="${camera_01}_link_camera" />
+    </joint>
+    <joint name="${camera_01}_camera_depth_joint" type="fixed">
+      <parent link="${camera_01}_link_camera" />
+      <child link="${camera_01}_camera_depth_frame" />
+      <origin xyz="0 0 0" rpy="0 0 0" />
+    </joint>
+    <joint name="${camera_01}_camera_depth_optical_joint" type="fixed">
+      <parent link="${camera_01}_camera_depth_frame" />
+      <child link="${camera_01}_camera_depth_optical_frame" />
+      <origin xyz="0 0 0" rpy="${-M_PI/2} 0 ${-M_PI/2}" />
+    </joint>
+    <joint name="${camera_01}_camera_color_joint" type="fixed">
+      <parent link="${camera_01}_link_camera" />
+      <child link="${camera_01}_camera_color_frame" />
+      <origin xyz="0 0.015 0" rpy="0 0 0" />
+    </joint>
+    <joint name="${camera_01}_camera_color_optical_joint" type="fixed">
+      <parent link="${camera_01}_camera_color_frame" />
+      <child link="${camera_01}_camera_color_optical_frame" />
+      <origin xyz="0 0 0" rpy="${-M_PI/2} 0 ${-M_PI/2}" />
+    </joint>
+    <joint name="${camera_01}_camera_left_ir_joint" type="fixed">
+      <parent link="${camera_01}_link_camera" />
+      <child link="${camera_01}_camera_left_ir_frame" />
+      <origin xyz="0 0 0" rpy="0 0 0" />
+    </joint>
+    <joint name="${camera_01}_camera_left_ir_optical_joint" type="fixed">
+      <parent link="${camera_01}_camera_left_ir_frame" />
+      <child link="${camera_01}_camera_left_ir_optical_frame" />
+      <origin xyz="0 0 0" rpy="${-M_PI/2} 0 ${-M_PI/2}" />
+    </joint>
+    <joint name="${camera_01}_camera_right_ir_joint" type="fixed">
+      <parent link="${camera_01}_link_camera" />
+      <child link="${camera_01}_camera_right_ir_frame" />
+      <origin xyz="0 -0.050 0" rpy="0 0 0" />
+    </joint>
+    <joint name="${camera_01}_camera_right_ir_optical_joint" type="fixed">
+      <parent link="${camera_01}_camera_right_ir_frame" />
+      <child link="${camera_01}_camera_right_ir_optical_frame" />
+      <origin xyz="0 0 0" rpy="${-M_PI/2} 0 ${-M_PI/2}" />
+    </joint>
+    <gazebo reference="${camera_01}_link_camera">
       <material>Gazebo/Black</material>
     </gazebo>
-   <gazebo reference="${prefix}link_camera">
+    <gazebo reference="${camera_01}_camera_depth_frame">
       <sensor name="cameradepth" type="depth">
         <camera name="camera">
@@ -54,32 +102,32 @@
         <always_on>1</always_on>
         <update_rate>30</update_rate>
+        <visualize>1</visualize>
+      </sensor>
+    </gazebo>
+    <gazebo reference="${camera_01}_camera_color_frame">
+      <sensor name="cameracolor" type="camera">
+        <camera name="camera">
+          <horizontal_fov>1.57</horizontal_fov>
+          <image>
+            <width>1280</width>
+            <height>720</height>
+            <format>RGB_INT8</format>
+          </image>
+          <clip>
+            <near>0.1</near>
+            <far>100</far>
+          </clip>
+          <noise>
+            <type>gaussian</type>
+            <mean>0.0</mean>
+            <stddev>0.007</stddev>
+          </noise>
+        </camera>
+        <always_on>1</always_on>
+        <update_rate>30</update_rate>
         <visualize>0</visualize>
       </sensor>
     </gazebo>
-    <gazebo reference="${prefix}link_camera">
-      <sensor name="cameracolor" type="camera">
-        <camera name="camera">
-          <horizontal_fov>1.57</horizontal_fov>
-          <image>
-            <width>1280</width>
-            <height>720</height>
-            <format>RGB_INT8</format>
-          </image>
-          <clip>
-            <near>0.1</near>
-            <far>100</far>
-          </clip>
-          <noise>
-            <type>gaussian</type>
-            <mean>0.0</mean>
-            <stddev>0.007</stddev>
-          </noise>
-        </camera>
-        <always_on>1</always_on>
-        <update_rate>30</update_rate>
-        <visualize>1</visualize>
-      </sensor>
-    </gazebo>
-    <gazebo reference="${prefix}link_camera">
+    <gazebo reference="${camera_01}_camera_left_ir_frame">
       <sensor name="cameraired1" type="camera">
         <camera name="camera">
@@ -105,5 +153,5 @@
       </sensor>
     </gazebo>
-    <gazebo reference="${prefix}link_camera">
+    <gazebo reference="${camera_01}_camera_right_ir_frame">
       <sensor name="cameraired2" type="camera">
         <camera name="camera">
@@ -143,4 +191,8 @@
         <infrared2TopicName>${camera_01}/infra2/image_raw</infrared2TopicName>
         <infrared2CameraInfoTopicName>${camera_01}/infra2/camera_info</infrared2CameraInfoTopicName>
+        <colorOpticalframeName>${camera_01}_camera_color_optical_frame</colorOpticalframeName>
+        <depthOpticalframeName>${camera_01}_camera_depth_optical_frame</depthOpticalframeName>
+        <infrared1OpticalframeName>${camera_01}_camera_left_ir_optical_frame</infrared1OpticalframeName>
+        <infrared2OpticalframeName>${camera_01}_camera_right_ir_optical_frame</infrared2OpticalframeName>
         <rangeMinDepth>0.3</rangeMinDepth>
         <rangeMaxDepth>3.0</rangeMaxDepth>

File: src/robot_descriptions/xarm6_description/urdf/camera/realsense.gazebo.xacro (robot description, xacro)
@@ -1,4 +1,5 @@
 <?xml version="1.0"?>
 <robot xmlns:xacro="http://ros.org/wiki/xacro">
+  <xacro:property name="camera_02" value="camera_gripper" />
   <xacro:macro name="realsense_gazebo" params="prefix:='' ">
     <gazebo reference="${prefix}camera_depth_frame">
@@ -22,5 +23,5 @@
         <always_on>1</always_on>
         <update_rate>30</update_rate>
-        <visualize>0</visualize>
+        <visualize>1</visualize>
       </sensor>
     </gazebo>
@@ -103,12 +104,12 @@
         <colorUpdateRate>30.0</colorUpdateRate>
         <infraredUpdateRate>30.0</infraredUpdateRate>
-        <depthTopicName>aligned_depth_to_color/image_raw</depthTopicName>
-        <depthCameraInfoTopicName>depth/camera_info</depthCameraInfoTopicName>
-        <colorTopicName>color/image_raw</colorTopicName>
-        <colorCameraInfoTopicName>color/camera_info</colorCameraInfoTopicName>
-        <infrared1TopicName>infra1/image_raw</infrared1TopicName>
+        <depthTopicName>${camera_02}/depth/image_raw</depthTopicName>
+        <depthCameraInfoTopicName>${camera_02}/depth/camera_info</depthCameraInfoTopicName>
+        <colorTopicName>${camera_02}/color/image_raw</colorTopicName>
+        <colorCameraInfoTopicName>${camera_02}/color/camera_info</colorCameraInfoTopicName>
+        <infrared1TopicName>${camera_02}/infra1/image_raw</infrared1TopicName>
         <infrared1CameraInfoTopicName>infra1/camera_info</infrared1CameraInfoTopicName>
-        <infrared2TopicName>infra2/image_raw</infrared2TopicName>
-        <infrared2CameraInfoTopicName>infra2/camera_info</infrared2CameraInfoTopicName>
+        <infrared2TopicName>${camera_02}/infra2/image_raw</infrared2TopicName>
+        <infrared2CameraInfoTopicName>${camera_02}/infra2/camera_info</infrared2CameraInfoTopicName>
         <colorOpticalframeName>camera_color_optical_frame</colorOpticalframeName>
         <depthOpticalframeName>camera_depth_optical_frame</depthOpticalframeName>
@@ -118,5 +119,5 @@
         <rangeMaxDepth>3.0</rangeMaxDepth>
         <pointCloud>true</pointCloud>
-        <pointCloudTopicName>depth/color/points</pointCloudTopicName>
+        <pointCloudTopicName>${camera_02}/depth/color/points</pointCloudTopicName>
         <pointCloudCutoff>0.3</pointCloudCutoff>
       </plugin>

File: src/robot_descriptions/xarm6_description/urdf/xarm_device_macro.xacro (robot description, xacro)
@@ -193,5 +193,5 @@
     <xacro:if value="${use_gazebo_camera}">
       <xacro:include filename="$(find xarm6_description)/urdf/camera/camera.gazebo.xacro" />
-      <xacro:camera_gazebo prefix="${prefix}" />
+      <xacro:camera_gazebo prefix="${prefix}"/>
     </xacro:if>
     <xacro:device_macro_end />
